File: pcb/Pinky3.kicad_pcb (KiCad board)
At the start: 2 copper layers, 137 x 100.9 mm, 67 parts, among them J1 MJ-4PP-9, P1 i2c-pin, P2 i2c-pin, SW1 RESET_SW, SW10 SW_PUSH, SW11 SW_PUSH, SW12 SW_PUSH, SW13 SW_PUSH, SW14 SW_PUSH, SW15 SW_PUSH, SW16 SW_PUSH, SW17 SW_PUSH, SW18 SW_PUSH, SW19 SW_PUSH, SW2 SW_PUSH, SW20 SW_PUSH, SW21 SW_PUSH, SW22 SW_PUSH, SW23 SW_PUSH, SW24 SW_PUSH, SW25 SW_PUSH, SW26 SW_PUSH, SW3 SW_PUSH, SW4 SW_PUSH, SW5 SW_PUSH, SW6 SW_PUSH, SW7 SW_PUSH, SW8 SW_PUSH, SW9 SW_PUSH, U1 ProMicro

Commit message: full update
Parts:
- removed the D22 at (164.3, 82.8)
- removed G*** (x2): LOGO, lib:pinky3
- removed the SW23 at (164.3, 74.8)
- added D7: D, kbd:D3_TH_SMD, F.Cu at (164.2, 83.5)
- added SW7: Rotary_Encoder_Switch, kbd:RotaryEncoder_Alps_EC11E-Switch_Vertical_H20mm-keebio_modified, F.Cu at (164.3, 74.8)
- JP1: footprint kbd:JP -> kbd:JPC2
- SW23: renamed from SW14; footprint kbd:Choc_Hotswap -> kbd:CherryMX_Choc_Hotswap
- SW24: renamed from SW18; footprint kbd:Choc_Hotswap -> kbd:CherryMX_Choc_Hotswap
- SW25: renamed from SW22; footprint kbd:Choc_Hotswap -> kbd:CherryMX_Choc_Hotswap
- SW26: footprint kbd:Choc_Hotswap -> kbd:CherryMX_Choc_Hotswap
- turned SW23 to 0 degrees
- turned SW24 to 350 degrees
- turned SW25 to 340 degrees
- turned SW26 to 330 degrees
- renumbered D8 to D10, D15 to D12, D19 to D13, D23 to D14, D3 to D15, D6 to D16, D9 to D17, D12 to D18, D16 to D19, D4 to D2, D24 to D21, D13 to D22, D17 to D23, D21 to D24, D7 to D3, D10 to D4, D14 to D5, D18 to D6, D2 to D8, D5 to D9, SW2 to SW1, SW9 to SW10, SW12 to SW11, SW16 to SW12, SW20 to SW13, SW24 to SW14, SW1 to SW15, SW4 to SW16, SW7 to SW17, SW10 to SW18, SW13 to SW19, SW5 to SW2, SW17 to SW20, SW25 to SW22, SW8 to SW3, SW11 to SW4, SW15 to SW5, SW19 to SW6, SW3 to SW8, SW6 to SW9
Connections:
- net col6 renamed SW7A
- J1 pad A: Net-(J1-PadA) -> VCC
- P1 pad 1: Net-(J1-PadA) -> VCC
- U1 pad 11: Net-(U1-Pad11) -> enc1
- U1 pad 12: Net-(U1-Pad12) -> enc2
Routing:
- net enc2: track 0.00 -> 174.3 mm
- net enc1: track 0.00 -> 161.9 mm
- net VCC: track 147.1 -> 234.8 mm, vias 1 -> 2
- net Net-(J1-PadA): track 87.8 -> 0.00 mm, vias 1 -> 0
- net GND: track 175.2 -> 210.8 mm, vias 50 -> 45
- net Net-(D25-Pad2): track 36.6 -> 57.1 mm
- net col5: track 242.4 -> 262.7 mm
- net col4: track 226.4 -> 245.2 mm
- net Net-(D22-Pad2) (its old number): track 18.4 -> 0.00 mm
- net Net-(U1-Pad12): track 17.1 -> 0.00 mm
- net Net-(U1-Pad11): track 17.1 -> 0.00 mm
- net SW7B: track 0.00 -> 16.8 mm
- net col3: track 214.8 -> 228.2 mm
- net Net-(D22-Pad2): track 35.3 -> 43.9 mm
- net SW7A: track 250.7 -> 258.5 mm, vias 6 -> 5
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Other:
- board text added: "designed by @tamanishi"
- board text removed: "ver. 1.0 designed by @tamanishi"
