File: pcb/Pinky3.sch (KiCad schematic (older format))
At the start: 58 parts, among them J1 MJ-4PP-9, P1 i2c-pin, P2 i2c-pin, SW1 RESET_SW, SW10 SW_PUSH, SW11 SW_PUSH, SW12 SW_PUSH, SW13 SW_PUSH, SW14 SW_PUSH, SW15 SW_PUSH, SW16 SW_PUSH, SW17 SW_PUSH, SW18 SW_PUSH, SW19 SW_PUSH, SW2 SW_PUSH, SW20 SW_PUSH, SW21 SW_PUSH, SW22 SW_PUSH, SW23 SW_PUSH, SW24 SW_PUSH, SW25 SW_PUSH, SW26 SW_PUSH, SW3 SW_PUSH, SW4 SW_PUSH, SW5 SW_PUSH, SW6 SW_PUSH, SW7 SW_PUSH, SW8 SW_PUSH, SW9 SW_PUSH, U1 ProMicro

Commit message: full update
Parts:
- removed D22: D, kbd:D3_TH_SMD, symbol Device:D
- removed SW23: SW_PUSH, kbd:CherryMX_Hotswap, symbol Pinky3-rescue:SW_PUSH-kbd
- added D7: D, kbd:D3_TH_SMD, symbol Device:D
- added SW7: Rotary_Encoder_Switch, kbd:RotaryEncoder_Alps_EC11E-Switch_Vertical_H20mm-keebio_modified, symbol Device:Rotary_Encoder_Switch
- SW23: renamed from SW14; footprint kbd:Choc_Hotswap -> kbd:CherryMX_Choc_Hotswap
- SW24: renamed from SW18; footprint kbd:Choc_Hotswap -> kbd:CherryMX_Choc_Hotswap
- SW25: renamed from SW22; footprint kbd:Choc_Hotswap -> kbd:CherryMX_Choc_Hotswap
- SW26: footprint kbd:Choc_Hotswap -> kbd:CherryMX_Choc_Hotswap
- renumbered D8 to D10, D15 to D12, D19 to D13, D23 to D14, D3 to D15, D6 to D16, D9 to D17, D12 to D18, D16 to D19, D4 to D2, D24 to D21, D13 to D22, D17 to D23, D21 to D24, D7 to D3, D10 to D4, D14 to D5, D18 to D6, D2 to D8, D5 to D9, SW2 to SW1, SW9 to SW10, SW12 to SW11, SW16 to SW12, SW20 to SW13, SW24 to SW14, SW1 to SW15, SW4 to SW16, SW7 to SW17, SW10 to SW18, SW13 to SW19, SW5 to SW2, SW17 to SW20, SW25 to SW22, SW8 to SW3, SW11 to SW4, SW15 to SW5, SW19 to SW6, SW3 to SW8, SW6 to SW9
Connections:
- net GND: now also SW7.C
- net VCC: now also J1.A, P1.1 (Pin_1)
- net row0: now also D7.1 (K)
- net enc1: now reaches U1.11 (B4)
- net enc1: now also SW7.A
- net enc2: now reaches U1.12 (B5)
- net enc2: now also SW7.B
- net col6 renamed SW7A
- net SW7A: now also SW7.S1
- new net SW7B: D7.2 (A), SW7.S2
- no-connect marks 5 -> 3
Other:
- moved on the sheet: D1, D10, D11, D12, D13, D14, D15, D16, D17, D18, D19, D2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
